File: PCB Design/Left/Keyboard - Left.sch (KiCad schematic (older format))
At the start: 129 parts, among them J1 AudioJack4, U1 ProMicroEliteC

Commit message: reworking pcb
Parts:
- J1: footprint Connector_Audio:Jack_3.5mm_PJ320D_Horizontal -> Keebio-Parts:TRRS-PJ-320A
Changed lines of the file:
@@
 EESchema Schematic File Version 4
-LIBS:Keyboard-cache
+LIBS:Keyboard - Left-cache
 EELAYER 30 0
 EELAYER END
@@
 F 0 "J1" H 1857 8275 50  0000 C CNN
 F 1 "AudioJack4" H 1857 8184 50  0000 C CNN
-F 2 "Connector_Audio:Jack_3.5mm_PJ320D_Horizontal" H 1900 7950 50  0001 C CNN
+F 2 "Keebio-Parts:TRRS-PJ-320A" H 1900 7950 50  0001 C CNN
 F 3 "~" H 1900 7950 50  0001 C CNN
 	1    1900 7950

Commit message: reworking PCB
Connections:
- net Col10: now also U1.28 (PF1); no longer U1.17 (A0/PF7)
- net Col11: now also U1.27 (PC7); no longer U1.18 (A1/PF6)
- net Col12: now also U1.26 (PD5); no longer U1.19 (A2/PF5)
- net Col5: now also U1.16 (15/PB1); no longer U1.8 (5/PC6)
- net Col6: now also U1.15 (14/PB3); no longer U1.13 (10/PB6)
- net Col8: now also U1.13 (10/PB6); no longer U1.15 (14/PB3)
- net Col9: now also U1.29 (PF0); no longer U1.16 (15/PB1)
- net Data1: now also R1.2; no longer R2.2
- net Data2: now also R2.2; no longer R1.2
- net RowA: now also U1.8 (5/PC6); no longer U1.20 (A3/PF4)
- net RowB: now also U1.25 (PB7); no longer U1.29 (PF0)
- net RowC: now also U1.17 (A0/PF7); no longer U1.28 (PF1)
- net RowD: now also U1.18 (A1/PF6); no longer U1.27 (PC7)
- net RowE: now also U1.19 (A2/PF5); no longer U1.26 (PD5)
- net RowF: now also U1.20 (A3/PF4); no longer U1.25 (PB7)
Changed lines of the file:
@@
 Text GLabel 5650 7950 0    50   Input ~ 0
 Data2
+Text GLabel 5650 8250 0    50   Input ~ 0
+RowA
+Text GLabel 5850 9000 3    50   Input ~ 0
+RowB
+Text GLabel 6550 8250 2    50   Input ~ 0
+RowC
+Text GLabel 6550 8150 2    50   Input ~ 0
+RowD
+Text GLabel 6550 8050 2    50   Input ~ 0
+RowE
 Text GLabel 6550 7950 2    50   Input ~ 0
-RowA
-Text GLabel 6250 9000 3    50   Input ~ 0
-RowB
-Text GLabel 6150 9000 3    50   Input ~ 0
-RowC
-Text GLabel 6050 9000 3    50   Input ~ 0
-RowD
-Text GLabel 5950 9000 3    50   Input ~ 0
-RowE
-Text GLabel 5850 9000 3    50   Input ~ 0
 RowF
 Text GLabel 5650 8650 0    50   Input ~ 0
@@
 Text GLabel 5650 8350 0    50   Input ~ 0
 Col4
-Text GLabel 5650 8250 0    50   Input ~ 0
+Text GLabel 6550 8350 2    50   Input ~ 0
 Col5
-Text GLabel 6550 8650 2    50   Input ~ 0
+Text GLabel 6550 8450 2    50   Input ~ 0
 Col6
 Text GLabel 6550 8550 2    50   Input ~ 0
 Col7
-Text GLabel 6550 8450 2    50   Input ~ 0
+Text GLabel 6550 8650 2    50   Input ~ 0
 Col8
-Text GLabel 6550 8350 2    50   Input ~ 0
+Text GLabel 6250 9000 3    50   Input ~ 0
 Col9
-Text GLabel 6550 8250 2    50   Input ~ 0
+Text GLabel 6150 9000 3    50   Input ~ 0
 Col10
-Text GLabel 6550 8150 2    50   Input ~ 0
+Text GLabel 6050 9000 3    50   Input ~ 0
 Col11
-Text GLabel 6550 8050 2    50   Input ~ 0
+Text GLabel 5950 9000 3    50   Input ~ 0
 Col12
 Text GLabel 6550 7750 2    50   Input ~ 0
@@
 	0    -1   -1   0
 $EndComp
+Text GLabel 1350 7250 0    50   Input ~ 0
+Data1
 Text GLabel 1900 7250 0    50   Input ~ 0
-Data1
-Text GLabel 1350 7250 0    50   Input ~ 0
 Data2
 $EndSCHEMATC
