File: PCB Design/Left/Keyboard - Left.kicad_pcb (KiCad board)
At the start: 2 copper layers, 257.2 x 133.4 mm, 129 parts, among them J1 AudioJack4, U1 ProMicroEliteC

Commit message: reworking pcb
Parts:
- D_A1, D_A10, D_A11, D_A12, D_A2, D_A3, D_A4, D_A5, D_A7, D_A8, D_A9, D_B1, D_B10, D_B11, D_B12, D_B2, D_B3, D_B4, D_B5, D_B6, D_B7, D_B8, D_B9, D_C1, D_C10, D_C11, D_C2, D_C3, D_C4, D_C5, D_C6, D_C7, D_C8, D_C9, D_D1, D_D10, D_D11, D_D2, D_D3, D_D5, D_D6, D_D7, D_D8, D_D9, D_E1, D_E10, D_E11, D_E2, D_E3, D_E4, D_E5, D_E6, D_E7, D_E8, D_E9, D_F1, D_F10, D_F3, D_F5, D_F6, D_F7, D_F8, R1, R2: moved to F.Cu
- J1: footprint Connector_Audio:Jack_3.5mm_PJ320D_Horizontal -> Keebio-Parts:TRRS-PJ-320A; moved to B.Cu
- U1: moved to B.Cu
- moved D_D3 22.0 mm to (85.3, 116.3)
- moved D_E3 20.4 mm to (85.6, 131.3)
- moved D_C3 20.2 mm to (85.6, 92.7)
- moved D_B2 19.8 mm to (67.1, 70.6)
- moved D_C2 19.8 mm to (67.1, 89.7)
- moved D_C1 19.6 mm to (47.8, 89.7)
- moved D_D1 19.6 mm to (47.8, 108.7)
- moved D_C4 19.4 mm to (104.6, 99.3)
- moved D_D2 19.3 mm to (66.5, 108.7)
- moved D_E2 19.3 mm to (66.5, 127.8)
- moved D_B1 19.3 mm to (47.5, 70.6)
- moved D_E1 19.3 mm to (47.5, 127.8)
- moved D_E4 19.3 mm to (104.6, 137.2)
- moved D_B4 19.1 mm to (104.4, 70.6)
- moved D_B3 19.1 mm to (85.3, 70.6)
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Routing:
- net RowE: track 466.0 -> 0.00 mm
- net RowD: track 425.6 -> 0.00 mm
- net RowC: track 418.5 -> 0.00 mm
- net RowF: track 417.6 -> 0.00 mm
- net RowB: track 405.9 -> 0.00 mm
- net RowA: track 346.7 -> 7.40 mm
- net Col12: track 260.3 -> 32.5 mm
- net Col11: track 307.0 -> 99.5 mm
- net Col10: track 303.4 -> 117.6 mm
- net Col9: track 260.1 -> 95.6 mm
- net Data1: track 158.7 -> 0.00 mm
- net Data2: track 150.8 -> 0.00 mm
- net Col8: track 260.9 -> 117.6 mm
- net Col2: track 248.6 -> 106.8 mm
- net Col4: track 287.3 -> 152.9 mm
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- removed copper zone on B.Cu, net GND
Other:
- board outline removed

Commit message: reworking PCB
Parts:
- moved U1 0.57 mm to (37.8, 47.0)
- moved SW_A5 0.35 mm to (126.2, 35.7)
Connections:
- R1 pad 2: Data2 -> Data1
- R2 pad 2: Data1 -> Data2
- U1 pad 13: Col6 -> Col8
- U1 pad 15: Col8 -> Col6
- U1 pad 16: Col9 -> Col5
- U1 pad 17: Col10 -> RowC
- U1 pad 18: Col11 -> RowD
- U1 pad 19: Col12 -> RowE
- U1 pad 20: RowA -> RowF
- U1 pad 25: RowF -> RowB
- U1 pad 26: RowE -> Col12
- U1 pad 27: RowD -> Col11
- U1 pad 28: RowC -> Col10
- U1 pad 29: RowB -> Col9
- U1 pad 8: Col5 -> RowA
Routing:
- net RowE: track 0.00 -> 320.2 mm
- net RowF: track 0.00 -> 304.5 mm
- net RowD: track 0.00 -> 285.5 mm
- net RowC: track 0.00 -> 267.0 mm
- net Col12: track 32.5 -> 299.3 mm
- net Col11: track 99.5 -> 345.8 mm
- net RowB: track 0.00 -> 239.9 mm
- net Col10: track 117.6 -> 344.1 mm
- net RowA: track 7.40 -> 227.3 mm
- net Col9: track 95.6 -> 301.7 mm
- net Col8: track 117.6 -> 303.8 mm
- net Col7: track 119.7 -> 291.5 mm
- net Data2: track 0.00 -> 120.4 mm
- net Data1: track 0.00 -> 117.0 mm
- net Col6: track 194.8 -> 250.8 mm
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Other:
- board outline added: 251.7 x 128.3 mm
