File: PCB Design/Right/Split Keyboard - Right.sch (KiCad schematic (older format))
At the start: 121 parts, among them J1 AudioJack4, U1 ProMicroEliteC

Commit message: Added Left information. Tweaks to right side
Parts:
- D_A1, D_A10, D_A11, D_A2, D_A3, D_A4, D_A5, D_A6, D_A7, D_A8, D_A9, D_B1, D_B10, D_B11, D_B2, D_B3, D_B4, D_B5, D_B6, D_B7, D_B8, D_B9, D_C1, D_C10, D_C11, D_C12, D_C2, D_C3, D_C4, D_C5, D_C6, D_C7, D_C8, D_C9, D_D10, D_D11, D_D4, D_D5, D_D6, D_D7, D_D8, D_D9, D_E10, D_E11, D_E2, D_E4, D_E6, D_E7, D_E8, D_E9, D_F1, D_F2, D_F3, D_F4, D_F5, D_F6, D_F7, D_F8, D_F9: footprint Diode_THT:D_DO-35_SOD27_P3.81mm_Vertical_AnodeUp -> combodiode:ComboDiode; symbol Split-Keyboard---Right-rescue:D-keyboard_parts -> keyboard_parts:D
- SW_A1, SW_A10, SW_A11, SW_A2, SW_A3, SW_A4, SW_A5, SW_A6, SW_A7, SW_A8, SW_A9, SW_B1, SW_B10, SW_B11, SW_B2, SW_B3, SW_B4, SW_B5, SW_B6, SW_B7, SW_B8, SW_B9, SW_C1, SW_C10, SW_C11, SW_C12, SW_C2, SW_C3, SW_C4, SW_C5, SW_C6, SW_C7, SW_C8, SW_C9, SW_D10, SW_D11, SW_D4, SW_D5, SW_D6, SW_D7, SW_D8, SW_D9, SW_E10, SW_E11, SW_E2, SW_E4, SW_E6, SW_E7, SW_E8, SW_E9, SW_F1, SW_F2, SW_F3, SW_F4, SW_F5, SW_F6, SW_F7, SW_F8, SW_F9, SW_R1: symbol Split-Keyboard---Right-rescue:SW_PUSH-keyboard_parts -> keyboard_parts:SW_PUSH

Commit message: reworking PCB
Parts:
- J1: footprint Connector_Audio:Jack_3.5mm_PJ320D_Horizontal -> Keebio-Parts:TRRS-PJ-320A
Changed lines of the file:
@@
 F 0 "J1" H 2557 5925 50  0000 C CNN
 F 1 "AudioJack4" H 2557 5834 50  0000 C CNN
-F 2 "Connector_Audio:Jack_3.5mm_PJ320D_Horizontal" H 2600 5600 50  0001 C CNN
+F 2 "Keebio-Parts:TRRS-PJ-320A" H 2600 5600 50  0001 C CNN
 F 3 "~" H 2600 5600 50  0001 C CNN
 	1    2600 5600

Commit message: Updated Right PCB
Parts:
- D_A1, D_A10, D_A11, D_A2, D_A3, D_A4, D_A5, D_A6, D_A7, D_A8, D_A9, D_B1, D_B10, D_B11, D_B2, D_B3, D_B4, D_B5, D_B6, D_B7, D_B8, D_B9, D_C1, D_C10, D_C11, D_C12, D_C2, D_C3, D_C4, D_C5, D_C6, D_C7, D_C8, D_C9, D_D10, D_D11, D_D4, D_D5, D_D6, D_D7, D_D8, D_D9, D_E10, D_E11, D_E2, D_E4, D_E6, D_E7, D_E8, D_E9, D_F1, D_F2, D_F3, D_F4, D_F5, D_F6, D_F7, D_F8, D_F9: symbol keyboard_parts:D -> Split-Keyboard---Right-rescue:D-keyboard_parts
- SW_A1, SW_A10, SW_A11, SW_A2, SW_A3, SW_A4, SW_A5, SW_A6, SW_A7, SW_A8, SW_A9, SW_B1, SW_B10, SW_B11, SW_B2, SW_B3, SW_B4, SW_B5, SW_B6, SW_B7, SW_B8, SW_B9, SW_C1, SW_C10, SW_C11, SW_C12, SW_C2, SW_C3, SW_C4, SW_C5, SW_C6, SW_C7, SW_C8, SW_C9, SW_D10, SW_D11, SW_D4, SW_D5, SW_D6, SW_D7, SW_D8, SW_D9, SW_E10, SW_E11, SW_E2, SW_E4, SW_E6, SW_E7, SW_E8, SW_E9, SW_F1, SW_F2, SW_F3, SW_F4, SW_F5, SW_F6, SW_F7, SW_F8, SW_F9, SW_R1: symbol keyboard_parts:SW_PUSH -> Split-Keyboard---Right-rescue:SW_PUSH-keyboard_parts
- U1: symbol Microcontroller:ProMicroEliteC -> Split-Keyboard---Right-rescue:ProMicroEliteC-Microcontroller
Connections:
- net Col1: now also U1.11 (8/PB4); no longer U1.18 (A1/PF6)
- net Col10: now also U1.12 (9/PB5); no longer U1.15 (14/PB3)
- net Col11: now also U1.10 (7/PE6); no longer U1.16 (15/PB1)
- net Col12: now also U1.9 (6/PD7); no longer U1.17 (A0/PF7)
- net Col2: now also U1.20 (A3/PF4); no longer U1.19 (A2/PF5)
- net Col3: now also U1.19 (A2/PF5); no longer U1.20 (A3/PF4)
- net Col4: now also U1.8 (5/PC6); no longer U1.26 (PD5)
- net Col5: now also U1.29 (PF0); no longer U1.27 (PC7)
- net Col7: now also U1.27 (PC7); no longer U1.29 (PF0)
- net Col8: now also U1.26 (PD5); no longer U1.13 (10/PB6)
- net Col9: now also U1.25 (PB7); no longer U1.14 (16/PB2)
- net RowA: now also U1.18 (A1/PF6); no longer U1.8 (5/PC6)
- net RowB: now also U1.17 (A0/PF7); no longer U1.9 (6/PD7)
- net RowC: now also U1.16 (15/PB1); no longer U1.7 (4/PD4)
- net RowD: now also U1.15 (14/PB3); no longer U1.10 (7/PE6)
- net RowE: now also U1.14 (16/PB2); no longer U1.11 (8/PB4)
- net RowF: now also U1.13 (10/PB6); no longer U1.12 (9/PB5)
